Commit message: added extra DOFs via extra URDF joints and reduction of task space. also 2ndary task to push blade towards Reye() to make its behavior more reasonable

File: urdf/sevenDOF_8_stat_tgt.urdf (robot description, URDF)
Before this commit: robot sevenDOF, 44 links, 43 joints
Links:
- added link tip-sliding
- added link tip-sliding-roll
- link cube: geometry collision box size=0.10 1.0 0.10; visual box size=0.1 1.0 0.1
Joints:
- added joint blade-length: type prismatic, parent tip, child tip-sliding, origin xyz=0 0 0 rpy=0 0 0, axis 0 1 0, limit lower=-0.5 upper=0.5 effort=1.0 velocity=1000000
- added joint blade-roll: type continuous, parent tip-sliding, child tip-sliding-roll, origin xyz=0 0 0 rpy=0 0 0, axis 0 1 0
