Commit message: Added single and double blade urdf

File: urdf/sevenDOF_double.urdf (robot description, URDF)
Before this commit: robot sevenDOF, 30 links, 29 joints
Links:
- removed link leftfinger
- removed link rightfinger
- removed link saber
- added link saber-left; visual cylinder length=1.0 radius=0.01
- added link saber-right; visual cylinder length=1.0 radius=0.01
- link handbase: geometry collision cylinder length=0.1 radius=0.01; visual cylinder length=0.1 radius=0.015
- link motor1: geometry collision cylinder length=0.2 radius=0.05; visual cylinder length=0.2 radius=0.04
- link motor2: geometry collision cylinder length=0.2 radius=0.05; visual sphere radius=0.08
- link motor3: geometry collision cylinder length=0.2 radius=0.05; visual cylinder length=0.2 radius=0.03
- link motor4: geometry collision cylinder length=0.2 radius=0.05; visual sphere radius=0.05
- link motor5: geometry collision cylinder length=0.1 radius=0.025; visual cylinder length=0.1 radius=0.015
- link motor6: geometry collision cylinder length=0.1 radius=0.025; visual sphere radius=0.04
- link motor7: geometry collision cylinder length=0.1 radius=0.025; visual sphere radius=0.03
- link mount1: geometry collision cylinder length=0.2 radius=0.02; visual cylinder length=0.298 radius=0.05
- link mount2: geometry collision cylinder length=0.2 radius=0.02; visual cylinder length=0.298 radius=0.05
- link mount3: geometry collision cylinder length=0.2 radius=0.02; visual cylinder length=0.198 radius=0.04
- link mount4: geometry collision cylinder length=0.2 radius=0.02; visual cylinder length=0.198 radius=0.04
- link mount5: geometry collision cylinder length=0.2 radius=0.02; visual cylinder length=0.198 radius=0.025
- link mount6: geometry collision cylinder length=0.2 radius=0.01; visual cylinder length=0.198 radius=0.025
- link palm: geometry visual cylinder length=0.1 radius=0.015
Joints:
- removed joint attach-leftfinger
- removed joint attach-rightfinger
- removed joint attach-saber
- added joint attach-saber-left: type fixed, parent tip, child saber-left
- added joint attach-saber-right: type fixed, parent tip, child saber-right

Commit message: Updated single and double urdf
Changed colors; unified visual and collision

File: urdf/sevenDOF_double.urdf (robot description, URDF)
Before this commit: robot sevenDOF, 29 links, 28 joints
Links:
- link handbase: geometry collision cylinder length=0.1 radius=0.015; visual cylinder length=0.1 radius=0.015
- link motor1: geometry collision cylinder length=0.2 radius=0.04; visual cylinder length=0.2 radius=0.04
- link motor2: geometry collision sphere radius=0.08; visual sphere radius=0.08
- link motor3: geometry collision cylinder length=0.2 radius=0.03; visual cylinder length=0.2 radius=0.03
- link motor4: geometry collision sphere radius=0.05; visual sphere radius=0.05
- link motor5: geometry collision cylinder length=0.1 radius=0.015; visual cylinder length=0.1 radius=0.015
- link motor6: geometry collision sphere radius=0.04; visual sphere radius=0.04
- link motor7: geometry collision sphere radius=0.03; visual sphere radius=0.03
- link mount1: geometry collision cylinder length=0.298 radius=0.05; visual cylinder length=0.298 radius=0.05
- link mount2: geometry collision cylinder length=0.298 radius=0.05; visual cylinder length=0.298 radius=0.05
- link mount3: geometry collision cylinder length=0.198 radius=0.04; visual cylinder length=0.198 radius=0.04
- link mount4: geometry collision cylinder length=0.198 radius=0.04; visual cylinder length=0.198 radius=0.04
- link mount5: geometry collision cylinder length=0.198 radius=0.025; visual cylinder length=0.198 radius=0.025
- link mount6: geometry collision cylinder length=0.198 radius=0.025; visual cylinder length=0.198 radius=0.025

File: urdf/sevenDOF_single.urdf (robot description, URDF)
Before this commit: robot sevenDOF, 27 links, 26 joints
Links:
- link handbase: geometry collision cylinder length=0.04 radius=0.015; visual cylinder length=0.04 radius=0.015
- link motor1: geometry collision cylinder length=0.2 radius=0.04; visual cylinder length=0.2 radius=0.04
- link motor2: geometry collision sphere radius=0.08; visual sphere radius=0.08
- link motor3: geometry collision cylinder length=0.2 radius=0.03; visual cylinder length=0.2 radius=0.03
- link motor4: geometry collision sphere radius=0.05; visual sphere radius=0.05
- link motor5: geometry collision cylinder length=0.1 radius=0.015; visual cylinder length=0.1 radius=0.015
- link motor6: geometry collision sphere radius=0.04; visual sphere radius=0.04
- link motor7: geometry collision sphere radius=0.03; visual sphere radius=0.03
- link mount1: geometry collision cylinder length=0.298 radius=0.05; visual cylinder length=0.298 radius=0.05
- link mount2: geometry collision cylinder length=0.298 radius=0.05; visual cylinder length=0.298 radius=0.05
- link mount3: geometry collision cylinder length=0.198 radius=0.04; visual cylinder length=0.198 radius=0.04
- link mount4: geometry collision cylinder length=0.198 radius=0.04; visual cylinder length=0.198 radius=0.04
- link mount5: geometry collision cylinder length=0.198 radius=0.025; visual cylinder length=0.198 radius=0.025
- link mount6: geometry collision cylinder length=0.198 radius=0.025; visual cylinder length=0.198 radius=0.025
