Commit message: Brought the updates on fake joints in sub-branch to main (previous version stored in beat_saber_old.py). Also improved graphics of cubes that show the direction types.

File: urdf/sevenDOF_8_stat_tgt_new.urdf (robot description, URDF)
Before this commit: robot sevenDOF, 27 links, 26 joints
Links:
- added link tip-sliding
- added link tip-sliding-roll
Joints:
- added joint blade-length: type prismatic, parent tip, child tip-sliding, origin xyz=0 0 0 rpy=0 0 0, axis 0 1 0, limit lower=-0.5 upper=0.5 effort=1.0 velocity=1000000
- added joint blade-roll: type continuous, parent tip-sliding, child tip-sliding-roll, origin xyz=0 0 0 rpy=0 0 0, axis 0 1 0
