Commit message: Added duo blade setup. Changed urdf file naming

File: urdf/sevenDOF.urdf (robot description, URDF)
Before this commit: robot sevenDOF, 36 links, 35 joints
Links:
- removed link cube
- removed link cube-xm
- removed link cube-xp
- removed link cube-ym
- removed link cube-yp
- removed link cube-zm
- removed link cube-zp
- removed link leftfinger
- removed link palm
- removed link rightfinger
- added link saber; visual cylinder length=1.0 radius=0.01
- link handbase: geometry collision cylinder length=0.04 radius=0.015; visual cylinder length=0.04 radius=0.015
- link motor1: geometry collision cylinder length=0.2 radius=0.04; visual cylinder length=0.2 radius=0.04
- link motor2: geometry collision sphere radius=0.08; visual sphere radius=0.08
- link motor3: geometry collision cylinder length=0.2 radius=0.03; visual cylinder length=0.2 radius=0.03
- link motor4: geometry collision sphere radius=0.05; visual sphere radius=0.05
- link motor5: geometry collision cylinder length=0.1 radius=0.015; visual cylinder length=0.1 radius=0.015
- link motor6: geometry collision sphere radius=0.04; visual sphere radius=0.04
- link motor7: geometry collision sphere radius=0.03; visual sphere radius=0.03
- link mount1: geometry collision cylinder length=0.298 radius=0.05; visual cylinder length=0.298 radius=0.05
- link mount2: geometry collision cylinder length=0.298 radius=0.05; visual cylinder length=0.298 radius=0.05
- link mount3: geometry collision cylinder length=0.198 radius=0.04; visual cylinder length=0.198 radius=0.04
- link mount4: geometry collision cylinder length=0.198 radius=0.04; visual cylinder length=0.198 radius=0.04
- link mount5: geometry collision cylinder length=0.198 radius=0.025; visual cylinder length=0.198 radius=0.025
- link mount6: geometry collision cylinder length=0.198 radius=0.025; visual cylinder length=0.198 radius=0.025
Joints:
- removed joint attach-cube
- removed joint attach-cube-xm
- removed joint attach-cube-xp
- removed joint attach-cube-ym
- removed joint attach-cube-yp
- removed joint attach-cube-zm
- removed joint attach-cube-zp
- removed joint attach-leftfinger
- removed joint attach-palm
- removed joint attach-rightfinger
- added joint attach-saber: type fixed, parent tip, child saber

File: urdf/sevenDOF_duo_vis.urdf (robot description, URDF)
Before this commit: robot sevenDOF, 29 links, 28 joints
Links:
- removed link saber
- removed link tip
- removed link tip-sliding
- removed link tip-sliding-roll
- added link palm, mass 0.05; visual cylinder length=0.1 radius=0.015
- added link saber-left; visual cylinder length=1.0 radius=0.01
- added link saber-right; visual cylinder length=1.0 radius=0.01
- added link tip-left
- added link tip-sliding-left
- added link tip-sliding-right
- added link tip-sliding-roll-left
- added link tip-sliding-roll-right
- added link vjoint-left; visual cylinder length=0.2 radius=0.03
- added link vjoint-right; visual cylinder length=0.2 radius=0.03
- link handbase: geometry collision cylinder length=0.1 radius=0.015; visual cylinder length=0.1 radius=0.015
Joints:
- removed joint attach-saber
- removed joint blade-length
- removed joint blade-roll
- removed joint final
- added joint attach-palm: type fixed, parent link7, child palm
- added joint attach-saber-left: type fixed, parent tip-left, child saber-left
- added joint attach-saber-right: type fixed, parent tip-left, child saber-right
- added joint attach-vjoint-left: type fixed, parent tip-sliding-roll-left, child vjoint-left
- added joint attach-vjoint-right: type fixed, parent tip-sliding-roll-right, child vjoint-right
- added joint blade-length-left: type prismatic, parent tip-left, child tip-sliding-left, origin xyz=0 0 0 rpy=0 0 0, axis 1 0 0, limit lower=-0.5 upper=0.5 effort=1.0 velocity=1000000
- added joint blade-length-right: type prismatic, parent tip-sliding-roll-left, child tip-sliding-right, origin xyz=0 0 0 rpy=0 0 0, axis 1 0 0, limit lower=-0.5 upper=0.5 effort=1.0 velocity=1000000
- added joint blade-roll-left: type continuous, parent tip-sliding-left, child tip-sliding-roll-left, origin xyz=0 0 0 rpy=0 0 0, axis 1 0 0
- added joint blade-roll-right: type continuous, parent tip-sliding-right, child tip-sliding-roll-right, origin xyz=0 0 0 rpy=0 0 0, axis 1 0 0
- added joint final-left: type fixed, parent link7, child tip-left, origin xyz=-0.5 0.1 0 rpy=0 0 0

File: urdf/sevenDOF_vis.urdf (robot description, URDF)
Before this commit: robot sevenDOF, 27 links, 26 joints
Links:
- added link tip-sliding
- added link tip-sliding-roll
- added link vjoint; visual cylinder length=0.2 radius=0.03
Joints:
- added joint attach-vjoint: type fixed, parent tip-sliding-roll, child vjoint
- added joint blade-length: type prismatic, parent tip, child tip-sliding, origin xyz=0 0 0 rpy=0 0 0, axis 0 1 0, limit lower=-0.5 upper=0.5 effort=1.0 velocity=1000000
- added joint blade-roll: type continuous, parent tip-sliding, child tip-sliding-roll, origin xyz=0 0 0 rpy=0 0 0, axis 0 1 0

Commit message: Final commit before submission
Improved beat_saber (single) by preventing the fictitious roller to spin around. The same improvement does not work well on the duo setup, so it is not used there. Also added the original version as beat_saber_og.py. This has the point-to-point goal without fictitious joints. Also small updates to urdf files.

File: urdf/sevenDOF.urdf (robot description, URDF)
Before this commit: robot sevenDOF, 27 links, 26 joints
Links:
- added link tip-sliding
- added link tip-sliding-roll
Joints:
- added joint blade-length: type prismatic, parent tip, child tip-sliding, origin xyz=0 0 0 rpy=0 0 0, axis 0 1 0, limit lower=-0.5 upper=0.5 effort=1.0 velocity=1000000
- added joint blade-roll: type continuous, parent tip-sliding, child tip-sliding-roll, origin xyz=0 0 0 rpy=0 0 0, axis 0 1 0

File: urdf/sevenDOF_duo.urdf (robot description, URDF)
Before this commit: robot sevenDOF, 29 links, 28 joints
Links:
- removed link tip
- added link tip-left
- added link tip-sliding-left
- added link tip-sliding-right
- added link tip-sliding-roll-left
- added link tip-sliding-roll-right
Joints:
- removed joint final
- added joint blade-length-left: type prismatic, parent tip-left, child tip-sliding-left, origin xyz=0 0 0 rpy=0 0 0, axis 1 0 0, limit lower=-0.5 upper=0.5 effort=1.0 velocity=1000000
- added joint blade-length-right: type prismatic, parent tip-sliding-roll-left, child tip-sliding-right, origin xyz=0 0 0 rpy=0 0 0, axis 1 0 0, limit lower=-0.5 upper=0.5 effort=1.0 velocity=1000000
- added joint blade-roll-left: type continuous, parent tip-sliding-left, child tip-sliding-roll-left, origin xyz=0 0 0 rpy=0 0 0, axis 1 0 0
- added joint blade-roll-right: type continuous, parent tip-sliding-right, child tip-sliding-roll-right, origin xyz=0 0 0 rpy=0 0 0, axis 1 0 0
- added joint final-left: type fixed, parent link7, child tip-left, origin xyz=-0.5 0.1 0 rpy=0 0 0
- joint attach-saber-left: parent tip -> tip-left
- joint attach-saber-right: parent tip -> tip-left
